File: Hardware/MotorDrivers/MS8313/MS8313.kicad_sch (KiCad schematic)
At the start: 0 parts

Commit message: DRV8313 schematic done
Parts:
- added C1, C2, C3: C, symbol Device:C
- added C4: C_Polarized, symbol Device:C_Polarized
- added R1, R2, R3, R4, R5, R6, R7, R8: R, symbol Device:R
- added U1: MS8313, SpaghettiLAB:HTSSOP-28_L9.7-W4.4-P0.65-LS6.4-BL-EP, symbol SpaghettiLab:MS8313
- added U2, U3, U4: INA241A1xDDF, Package_TO_SOT_SMD:SOT-23-8, symbol Amplifier_Current:INA241A1xDDF
Connections:
- new net: U2.2 (GND), U2.4 (GND)
- new net: U3.2 (GND), U3.4 (GND)
- new net: U4.2 (GND), U4.4 (GND)
