File: Hardware/Core/RP2350-Core/RP2350-Core.kicad_pcb (KiCad board)
At the start: 4 copper layers, 66.8 x 65.6 mm, 87 parts, among them CN10 PR5L4015-5P-C-F, CN11 PR5L4015-5P-C-F, CN7 PR5L4015-5P-C-F, CN8 PR5L4015-5P-C-F, CN9 PR5L4015-5P-C-F, J2 Conn_02x05_Counter_Clockwise, J4 Conn_02x05_Counter_Clockwise, J5 Conn_02x05_Counter_Clockwise, J7 SWD, Q2 2N7002, Q3 2N7002, SW1 TS-1187A-B-A-B, SW2 TS-1187A-B-A-B, U19 W25Q16JVSNIQ, U2 AP2112K-3.3, U3 LM66200DRLR, U35 PR5L5015-5P-C-H, U36 PR5L5015-5P-C-H, U37 PR5L5015-5P-C-H, U38 PR5L5015-5P-C-H, U39 PR5L5015-5P-C-H, U4 RP2350A, Y1 Crystal

Commit message: Started routing and fixed flex label in core rp2350
Other:
- board text added: "FLEX3"
Changed lines of the file:
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@@
 				(font
 					(size 1.27 1.27)
+					(thickness 0.15)
 				)
 			)
@@
 				(font
 					(size 1.27 1.27)
+					(thickness 0.15)
 				)
 			)
@@
 				(font
 					(size 1.27 1.27)
+					(thickness 0.15)
 				)
 			)
@@
 			(at 0 4 134)
 			(layer "F.Fab")
+			(hide yes)
 			(effects
 				(font
@@
 				(font
 					(size 1.27 1.27)
+					(thickness 0.15)
 				)
 				(justify mirror)
@@
 				(font
 					(size 1.27 1.27)
+					(thickness 0.15)
 				)
 				(justify mirror)
@@
 				(font
 					(size 1.27 1.27)
+					(thickness 0.15)
 				)
 				(justify mirror)
@@
 				(font
 					(size 1.27 1.27)
+					(thickness 0.15)
 				)
 				(justify mirror)
@@
 		)
 	)
-	(gr_text "FLEX5"
+	(gr_text "FLEX3"
 		(at 72.78 91.05 0)
 		(layer "B.SilkS")
