File: Hardware/motion/salsa-AS5600-encoder/AS5600-encoder/as5600.kicad_pcb (KiCad board)
At the start: 2 copper layers, 66.8 x 65.6 mm, 52 parts, among them CN10 PR5L4015-5P-C-F, CN11 PR5L4015-5P-C-F, CN7 PR5L4015-5P-C-F, CN8 PR5L4015-5P-C-F, CN9 PR5L4015-5P-C-F, J1 Conn_01x04_Socket, U1 AS5600-ASOT, U35 PR5L5015-5P-C-H, U36 PR5L5015-5P-C-H, U37 PR5L5015-5P-C-H, U38 PR5L5015-5P-C-H, U39 PR5L5015-5P-C-H

Commit message: finished as5600 with some connector fix
Parts:
- added J3: Conn_01x04_Pin, Connector_PinHeader_2.54mm:PinHeader_1x04_P2.54mm_Vertical, F.Cu at (177.7, 137.3)
- J1: footprint Connector_JST:JST_GH_SM04B-GHS-TB_1x04-1MP_P1.25mm_Horizontal -> SpaghettiLAB:CONN-SMD_BM04B-SRSS-TB
- moved J1 0.99 mm to (181.3, 142.1), turned to 180 degrees
Routing:
- net +3.3V: track 62.4 -> 65.7 mm
- net /~{RESET}: track 89.9 -> 90.8 mm
