File: Hardware/motion/salsa-AS5600-encoder/AS5600-encoder/as5600.kicad_sch (KiCad schematic)
At the start: 19 parts, among them CN10 PR5L4015-5P-C-F, CN11 PR5L4015-5P-C-F, CN7 PR5L4015-5P-C-F, CN8 PR5L4015-5P-C-F, CN9 PR5L4015-5P-C-F, J1 Conn_01x04_Socket, U1 AS5600-ASOT, U35 PR5L5015-5P-C-H, U36 PR5L5015-5P-C-H, U37 PR5L5015-5P-C-H, U38 PR5L5015-5P-C-H, U39 PR5L5015-5P-C-H

Commit message: finished as5600 with some connector fix
Parts:
- added J3: Conn_01x04_Pin, Connector_PinHeader_2.54mm:PinHeader_1x04_P2.54mm_Vertical, symbol Connector:Conn_01x04_Pin
- J1: footprint Connector_JST:JST_GH_SM04B-GHS-TB_1x04-1MP_P1.25mm_Horizontal -> SpaghettiLAB:CONN-SMD_BM04B-SRSS-TB
Connections:
- net +3.3V: now also J3.2 (Pin_2)
- net GND: now also J3.1 (Pin_1)
- net ID: now also J3.3 (Pin_3)
- net ~{RESET}: now also J3.4 (Pin_4)
