File: Hardware/backbone/Backbone.kicad_pcb (KiCad board)
At the start: 4 copper layers, 31.3 x 67.7 mm, 83 parts, among them J1 RESET, J10 CORE_A, J11 MOUNT, J13 FIELD_B, J14 FIELD_A, J15 UART PROG, J2 FROM_PREVIOUS, J4 FROM_PREVIOUS, J5 CONN_A, J6 BOOTLOADER, J7 CONN_B, J8 CORE_B, J9 TO NEXT, Q2 AO3401A, U11 470nH DCR=450m, U13 470nH DCR=450m, U15 ST25R200, U17 BLM18PG471SZ1D, U2 SN65HVD230DR, U4 AP2112K-3.3TRG1, U5 ESP32-C3-MINI-1-H4X, U8 G3VM-61VY3, U9 SN74AHCT1G14DCKR, X1 NX2016SA 27.12MHz

Commit message: added label in silkscreen for backbone board and core board
Parts:
- moved C12 1.20 mm to (161.8, 97.1)
- moved TP20 0.33 mm to (157.1, 92.8)
Routing:
- net GND: track 98.4 -> 102.8 mm, vias 17 -> 23
Other:
- outline, holes or cut-outs redrawn
- board text added: "5v"
- board text added: "BACKBONE"
- board text added: "BOARD"
- board text added: "DUMMY"
- board text added: "ESP32-C3"
- board text added: "FIELD"
- board text added: "FROM OUTSIDE"
- board text added: "MCU"
- board text added: "NFC"
- board text added: "a0"
- board text added: "a1"
- board text added: "a2"
- board text added: "a3"
- board text added: "boot"
- board text added: "canH"
- board text added: "canL"
- board text added: "canRx"
- board text added: "canTx"
- board text added: "cs"
- board text added: "en"
- board text added: "gnd"
- board text added: "in"
- board text added: "irq"
- board text added: "led1"
- board text added: "led2"
- board text added: "led3"
- board text added: "led4"
- board text added: "miso"
- board text added: "mosi"
- board text added: "out"
- board text added: "rst"
- board text added: "sck"
- board text added: "term"

Commit message: added commercial name to backbone
Other:
- board text added: "PLATE"
- board text removed: "BACKBONE"
Changed lines of the file:
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@@
 	)
 	(gr_line
-		(start 154.02 106.13)
-		(end 154.02 107.03)
-		(stroke
-			(width 0.1)
-			(type default)
-		)
-		(layer "B.SilkS")
-	)
-	(gr_line
-		(start 154.105 112.845)
-		(end 154.105 113.695)
-		(stroke
-			(width 0.1)
-			(type default)
-		)
-		(layer "B.SilkS")
-	)
-	(gr_line
-		(start 154.105 113.695)
-		(end 155.005 113.695)
-		(stroke
-			(width 0.1)
-			(type default)
-		)
-		(layer "B.SilkS")
-	)
-	(gr_line
-		(start 154.87 106.13)
-		(end 154.02 106.13)
-		(stroke
-			(width 0.1)
-			(type default)
-		)
-		(layer "B.SilkS")
-	)
-	(gr_line
-		(start 156.18 113.68)
-		(end 157.03 113.68)
-		(stroke
-			(width 0.1)
-			(type default)
-		)
-		(layer "B.SilkS")
-	)
-	(gr_line
-		(start 157.03 113.68)
-		(end 157.03 112.78)
-		(stroke
-			(width 0.1)
-			(type default)
-		)
-		(layer "B.SilkS")
-	)
-	(gr_line
-		(start 157.165 106.13)
-		(end 156.265 106.13)
-		(stroke
-			(width 0.1)
-			(type default)
-		)
-		(layer "B.SilkS")
-	)
-	(gr_line
-		(start 157.165 106.98)
-		(end 157.165 106.13)
+		(start 177.8 102.925)
+		(end 177.8 103.825)
+		(stroke
+			(width 0.1)
+			(type default)
+		)
+		(layer "B.SilkS")
+	)
+	(gr_line
+		(start 177.8 105.1)
+		(end 177.8 105.95)
+		(stroke
+			(width 0.1)
+			(type default)
+		)
+		(layer "B.SilkS")
+	)
+	(gr_line
+		(start 177.8 105.95)
+		(end 178.7 105.95)
+		(stroke
+			(width 0.1)
+			(type default)
+		)
+		(layer "B.SilkS")
+	)
+	(gr_line
+		(start 178.65 102.925)
+		(end 177.8 102.925)
+		(stroke
+			(width 0.1)
+			(type default)
+		)
+		(layer "B.SilkS")
+	)
+	(gr_line
+		(start 181.76 105.98)
+		(end 182.61 105.98)
+		(stroke
+			(width 0.1)
+			(type default)
+		)
+		(layer "B.SilkS")
+	)
+	(gr_line
+		(start 182.61 102.835)
+		(end 181.71 102.835)
+		(stroke
+			(width 0.1)
+			(type default)
+		)
+		(layer "B.SilkS")
+	)
+	(gr_line
+		(start 182.61 103.685)
+		(end 182.61 102.835)
+		(stroke
+			(width 0.1)
+			(type default)
+		)
+		(layer "B.SilkS")
+	)
+	(gr_line
+		(start 182.61 105.98)
+		(end 182.61 105.08)
 		(stroke
 			(width 0.1)
@@
 		)
 	)
-	(gr_text "BACKBONE"
-		(at 155.58 106.22 90)
+	(gr_text "PLATE"
+		(at 182.52 104.395 0)
 		(layer "B.SilkS" knockout)
 		(effects
@@
 	)
 	(gr_text "BOARD"
-		(at 156.94 106.22 90)
-		(layer "B.SilkS")
-		(effects
+		(at 182.52 105.755 0)
+		(layer "B.SilkS")
+		(effects
