File: Hardware/core/core/core.kicad_pcb (KiCad board)
At the start: 4 copper layers, 31.3 x 67.7 mm, 32 parts, among them J17 PROG, J18 USB_C_Receptacle_USB2.0_14P, J5 TO_NEXT, J7 TO_NEXT, J8 Conn_02x09_Odd_Even, SW1 RESET, SW2 BOOT, U10 SN74AHCT1G14DCKR, U19 ESP32-S3-MINI-1, U20 AP2112K-3.3TRG1, U21 SN65HVD230DR

Commit message: added commerciali label for core board
Other:
- board text added: "PLATE"
- board text removed: "CORE"
Changed lines of the file:
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@@
 		(capping no)
 		(filling no)
-		(zone_defaults)
 		(pcbplotparams
 			(layerselection 0x00000000_00000000_55555555_5755f5ff)
@@
 		(layer "F.SilkS")
 	)
-	(gr_line
-		(start 82.595 120.14)
-		(end 83.665 120.14)
-		(stroke
-			(width 0.1)
-			(type default)
-		)
-		(layer "F.SilkS")
-	)
-	(gr_line
-		(start 82.595 120.93)
-		(end 82.595 120.14)
-		(stroke
-			(width 0.1)
-			(type default)
-		)
-		(layer "F.SilkS")
-	)
-	(gr_line
-		(start 82.635 125.49)
-		(end 82.635 124.42)
-		(stroke
-			(width 0.1)
-			(type default)
-		)
-		(layer "F.SilkS")
-	)
-	(gr_line
-		(start 83.425 125.49)
-		(end 82.635 125.49)
-		(stroke
-			(width 0.1)
-			(type default)
-		)
-		(layer "F.SilkS")
-	)
 	(gr_rect
 		(start 84.04 131.31)
@@
 		(layer "F.SilkS")
 	)
-	(gr_line
-		(start 85.45 120.14)
-		(end 86.24 120.14)
-		(stroke
-			(width 0.1)
-			(type default)
-		)
-		(layer "F.SilkS")
-	)
 	(gr_rect
 		(start 86.05 110.79)
@@
 		(layer "F.SilkS")
 	)
-	(gr_line
-		(start 86.24 120.14)
-		(end 86.24 121.21)
-		(stroke
-			(width 0.1)
-			(type default)
-		)
-		(layer "F.SilkS")
-	)
-	(gr_line
-		(start 86.28 124.7)
-		(end 86.28 125.49)
-		(stroke
-			(width 0.1)
-			(type default)
-		)
-		(layer "F.SilkS")
-	)
-	(gr_line
-		(start 86.28 125.49)
-		(end 85.21 125.49)
-		(stroke
-			(width 0.1)
-			(type default)
-		)
-		(layer "F.SilkS")
-	)
 	(gr_rect
 		(start 86.74 133.42)
@@
 		(layer "B.SilkS")
 	)
+	(gr_line
+		(start 68.91 75.03)
+		(end 68.91 75.82)
+		(stroke
+			(width 0.1)
+			(type default)
+		)
+		(layer "B.SilkS")
+	)
+	(gr_line
+		(start 68.91 75.82)
+		(end 69.98 75.82)
+		(stroke
+			(width 0.1)
+			(type default)
+		)
+		(layer "B.SilkS")
+	)
+	(gr_line
+		(start 68.95 70.47)
+		(end 68.95 71.54)
+		(stroke
+			(width 0.1)
+			(type default)
+		)
+		(layer "B.SilkS")
+	)
+	(gr_line
+		(start 69.74 70.47)
+		(end 68.95 70.47)
+		(stroke
+			(width 0.1)
+			(type default)
+		)
+		(layer "B.SilkS")
+	)
+	(gr_line
+		(start 71.765 75.82)
+		(end 72.555 75.82)
+		(stroke
+			(width 0.1)
+			(type default)
+		)
+		(layer "B.SilkS")
+	)
+	(gr_line
+		(start 72.555 75.82)
+		(end 72.555 74.75)
+		(stroke
+			(width 0.1)
+			(type default)
+		)
+		(layer "B.SilkS")
+	)
+	(gr_line
+		(start 72.595 70.47)
+		(end 71.525 70.47)
+		(stroke
+			(width 0.1)
+			(type default)
+		)
+		(layer "B.SilkS")
+	)
+	(gr_line
+		(start 72.595 71.26)
+		(end 72.595 70.47)
+		(stroke
+			(width 0.1)
+			(type default)
+		)
+		(layer "B.SilkS")
+	)
 	(gr_arc
 		(start 67.085239 71.7)
@@
 		)
 	)
-	(gr_text "CORE"
-		(at 84.28 124.95 90)
+	(gr_text "TO BACKBONE"
+		(at 88.21 82.95 90)
 		(layer "F.SilkS" knockout)
 		(effects
@@
 		)
 	)
-	(gr_text "BOARD"
-		(at 85.98 125.38 90)
-		(layer "F.SilkS")
+	(gr_text "DUMMY"
+		(at 89.05 128.24 90)
+		(layer "F.SilkS" knockout)
 		(effects
 			(font
@@
 		)
 	)
-	(gr_text "TO BACKBONE"
-		(at 88.21 82.95 90)
+	(gr_text "ESP32-S3"
+		(at 89.22 106.57 90)
 		(layer "F.SilkS" knockout)
 		(effects
@@
 		)
 	)
-	(gr_text "DUMMY"
-		(at 89.05 128.24 90)
+	(gr_text "BOOT"
+		(at 71.16 113.9 270)
 		(layer "F.SilkS" knockout)
 		(effects
@@
 		)
 	)
-	(gr_text "ESP32-S3"
-		(at 89.22 106.57 90)
+	(gr_text "PROG"
+		(at 96.39 100.44 270)
 		(layer "F.SilkS" knockout)
 		(effects
@@
 		)
 	)
-	(gr_text "BOOT"
-		(at 71.16 113.9 270)
-		(layer "F.SilkS" knockout)
+	(gr_text "PLATE"
+		(at 70.595 70.81 90)
+		(layer "B.SilkS" knockout)
 		(effects
 			(font
@@
 				(bold yes)
 			)
-			(justify left bottom)
+			(justify left bottom mirror)
 		)
 	)
-	(gr_text "PROG"
-		(at 96.39 100.44 270)
-		(layer "F.SilkS" knockout)
+	(gr_text "BOARD"
+		(at 72.295 70.58 90)
+		(layer "B.SilkS")
 		(effects
 			(font
@@
 				(bold yes)
 			)
-			(justify left bottom)
+			(justify left bottom mirror)
 		)
 	)

Commit message: modified commercial name for core board
Other:
- board text added: "SPICE"
- board text removed: "PLATE"
Changed lines of the file:
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@@
 		)
 	)
-	(gr_text "PLATE"
+	(gr_text "SPICE"
 		(at 70.595 70.81 90)
 		(layer "B.SilkS" knockout)
